Commit message: localization of file names

File: example/Linker_hand_Sapien/urdf/linker_hand_l20_6_left.urdf (robot description, URDF)
Before this commit: robot linker_hand_l20_6_right, 27 links, 26 joints
Links:
- link base_link: geometry collision mesh filename=meshes/real_hand_l20_6_right/base_link.STL; visual mesh filename=meshes/real_hand_l20_6_right/base_link.STL
- link index_link0: geometry collision mesh filename=meshes/real_hand_l20_6_right/index_link0.STL; visual mesh filename=meshes/real_hand_l20_6_right/index_link0.STL
- link index_link1: geometry collision mesh filename=meshes/real_hand_l20_6_right/index_link1.STL; visual mesh filename=meshes/real_hand_l20_6_right/index_link1.STL
- link index_link2: geometry collision mesh filename=meshes/real_hand_l20_6_right/index_link2.STL; visual mesh filename=meshes/real_hand_l20_6_right/index_link2.STL
- link index_link3: geometry collision mesh filename=meshes/real_hand_l20_6_right/index_link3.STL; visual mesh filename=meshes/real_hand_l20_6_right/index_link3.STL
- link little_link0: geometry collision mesh filename=meshes/real_hand_l20_6_right/little_link0.STL; visual mesh filename=meshes/real_hand_l20_6_right/little_link0.STL
- link little_link1: geometry collision mesh filename=meshes/real_hand_l20_6_right/little_link1.STL; visual mesh filename=meshes/real_hand_l20_6_right/little_link1.STL
- link little_link2: geometry collision mesh filename=meshes/real_hand_l20_6_right/little_link2.STL; visual mesh filename=meshes/real_hand_l20_6_right/little_link2.STL
- link little_link3: geometry collision mesh filename=meshes/real_hand_l20_6_right/little_link3.STL; visual mesh filename=meshes/real_hand_l20_6_right/little_link3.STL
- link middle_link0: geometry collision mesh filename=meshes/real_hand_l20_6_right/middle_link0.STL; visual mesh filename=meshes/real_hand_l20_6_right/middle_link0.STL
- link middle_link1: geometry collision mesh filename=meshes/real_hand_l20_6_right/middle_link1.STL; visual mesh filename=meshes/real_hand_l20_6_right/middle_link1.STL
- link middle_link2: geometry collision mesh filename=meshes/real_hand_l20_6_right/middle_link2.STL; visual mesh filename=meshes/real_hand_l20_6_right/middle_link2.STL
- link middle_link3: geometry collision mesh filename=meshes/real_hand_l20_6_right/middle_link3.STL; visual mesh filename=meshes/real_hand_l20_6_right/middle_link3.STL
- link ring_link0: geometry collision mesh filename=meshes/real_hand_l20_6_right/ring_link0.STL; visual mesh filename=meshes/real_hand_l20_6_right/ring_link0.STL
- link ring_link1: geometry collision mesh filename=meshes/real_hand_l20_6_right/ring_link1.STL; visual mesh filename=meshes/real_hand_l20_6_right/ring_link1.STL
- link ring_link2: geometry collision mesh filename=meshes/real_hand_l20_6_right/ring_link2.STL; visual mesh filename=meshes/real_hand_l20_6_right/ring_link2.STL
- link ring_link3: geometry collision mesh filename=meshes/real_hand_l20_6_right/ring_link3.STL; visual mesh filename=meshes/real_hand_l20_6_right/ring_link3.STL
- link thumb_link0: geometry collision mesh filename=meshes/real_hand_l20_6_right/thumb_link0.STL; visual mesh filename=meshes/real_hand_l20_6_right/thumb_link0.STL
- link thumb_link1: geometry collision mesh filename=meshes/real_hand_l20_6_right/thumb_link1.STL; visual mesh filename=meshes/real_hand_l20_6_right/thumb_link1.STL
- link thumb_link2: geometry collision mesh filename=meshes/real_hand_l20_6_right/thumb_link2.STL; visual mesh filename=meshes/real_hand_l20_6_right/thumb_link2.STL
- link thumb_link3: geometry collision mesh filename=meshes/real_hand_l20_6_right/thumb_link3.STL; visual mesh filename=meshes/real_hand_l20_6_right/thumb_link3.STL
- link thumb_link4: geometry collision mesh filename=meshes/real_hand_l20_6_right/thumb_link4.STL; visual mesh filename=meshes/real_hand_l20_6_right/thumb_link4.STL

File: example/Linker_hand_Sapien/urdf/linker_hand_l20_6_right.urdf (robot description, URDF)
Before this commit: robot linker_hand_l20_6_right, 27 links, 26 joints
Links:
- link base_link: geometry collision mesh filename=meshes/real_hand_l20_6_right/base_link.STL; visual mesh filename=meshes/real_hand_l20_6_right/base_link.STL
- link index_link0: geometry collision mesh filename=meshes/real_hand_l20_6_right/index_link0.STL; visual mesh filename=meshes/real_hand_l20_6_right/index_link0.STL
- link index_link1: geometry collision mesh filename=meshes/real_hand_l20_6_right/index_link1.STL; visual mesh filename=meshes/real_hand_l20_6_right/index_link1.STL
- link index_link2: geometry collision mesh filename=meshes/real_hand_l20_6_right/index_link2.STL; visual mesh filename=meshes/real_hand_l20_6_right/index_link2.STL
- link index_link3: geometry collision mesh filename=meshes/real_hand_l20_6_right/index_link3.STL; visual mesh filename=meshes/real_hand_l20_6_right/index_link3.STL
- link little_link0: geometry collision mesh filename=meshes/real_hand_l20_6_right/little_link0.STL; visual mesh filename=meshes/real_hand_l20_6_right/little_link0.STL
- link little_link1: geometry collision mesh filename=meshes/real_hand_l20_6_right/little_link1.STL; visual mesh filename=meshes/real_hand_l20_6_right/little_link1.STL
- link little_link2: geometry collision mesh filename=meshes/real_hand_l20_6_right/little_link2.STL; visual mesh filename=meshes/real_hand_l20_6_right/little_link2.STL
- link little_link3: geometry collision mesh filename=meshes/real_hand_l20_6_right/little_link3.STL; visual mesh filename=meshes/real_hand_l20_6_right/little_link3.STL
- link middle_link0: geometry collision mesh filename=meshes/real_hand_l20_6_right/middle_link0.STL; visual mesh filename=meshes/real_hand_l20_6_right/middle_link0.STL
- link middle_link1: geometry collision mesh filename=meshes/real_hand_l20_6_right/middle_link1.STL; visual mesh filename=meshes/real_hand_l20_6_right/middle_link1.STL
- link middle_link2: geometry collision mesh filename=meshes/real_hand_l20_6_right/middle_link2.STL; visual mesh filename=meshes/real_hand_l20_6_right/middle_link2.STL
- link middle_link3: geometry collision mesh filename=meshes/real_hand_l20_6_right/middle_link3.STL; visual mesh filename=meshes/real_hand_l20_6_right/middle_link3.STL
- link ring_link0: geometry collision mesh filename=meshes/real_hand_l20_6_right/ring_link0.STL; visual mesh filename=meshes/real_hand_l20_6_right/ring_link0.STL
- link ring_link1: geometry collision mesh filename=meshes/real_hand_l20_6_right/ring_link1.STL; visual mesh filename=meshes/real_hand_l20_6_right/ring_link1.STL
- link ring_link2: geometry collision mesh filename=meshes/real_hand_l20_6_right/ring_link2.STL; visual mesh filename=meshes/real_hand_l20_6_right/ring_link2.STL
- link ring_link3: geometry collision mesh filename=meshes/real_hand_l20_6_right/ring_link3.STL; visual mesh filename=meshes/real_hand_l20_6_right/ring_link3.STL
- link thumb_link0: geometry collision mesh filename=meshes/real_hand_l20_6_right/thumb_link0.STL; visual mesh filename=meshes/real_hand_l20_6_right/thumb_link0.STL
- link thumb_link1: geometry collision mesh filename=meshes/real_hand_l20_6_right/thumb_link1.STL; visual mesh filename=meshes/real_hand_l20_6_right/thumb_link1.STL
- link thumb_link2: geometry collision mesh filename=meshes/real_hand_l20_6_right/thumb_link2.STL; visual mesh filename=meshes/real_hand_l20_6_right/thumb_link2.STL
- link thumb_link3: geometry collision mesh filename=meshes/real_hand_l20_6_right/thumb_link3.STL; visual mesh filename=meshes/real_hand_l20_6_right/thumb_link3.STL
- link thumb_link4: geometry collision mesh filename=meshes/real_hand_l20_6_right/thumb_link4.STL; visual mesh filename=meshes/real_hand_l20_6_right/thumb_link4.STL

File: example/Linker_hand_Sapien/urdf/linker_hand_l20_8_left.urdf (robot description, URDF)
Before this commit: robot l20_8_l, 27 links, 26 joints
Links:
- link base_link: geometry collision mesh filename=package://real_hand_pybullet/urdf/meshes/real_hand_l20_8_le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; visual mesh filename=package://real_hand_pybullet/urdf/meshes/real_hand_l20_8_le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
- link index_link0: geometry collision mesh filename=package://real_hand_pybullet/urdf/meshes/real_hand_l20_8_le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; visual mesh filename=package://real_hand_pybullet/urdf/meshes/real_hand_l20_8_le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
- link index_link1: geometry collision mesh filename=package://real_hand_pybullet/urdf/meshes/real_hand_l20_8_le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; visual mesh filename=package://real_hand_pybullet/urdf/meshes/real_hand_l20_8_le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
- link index_link2: geometry collision mesh filename=package://real_hand_pybullet/urdf/meshes/real_hand_l20_8_le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; visual mesh filename=package://real_hand_pybullet/urdf/meshes/real_hand_l20_8_le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
- link index_link3: geometry collision mesh filename=package://real_hand_pybullet/urdf/meshes/real_hand_l20_8_le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; visual mesh filename=package://real_hand_pybullet/urdf/meshes/real_hand_l20_8_le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
- link index_link4: geometry collision mesh filename=package://real_hand_pybullet/urdf/meshes/real_hand_l20_8_le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; visual mesh filename=package://real_hand_pybullet/urdf/meshes/real_hand_l20_8_le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
- link little_link0: geometry collision mesh filename=package://real_hand_pybullet/urdf/meshes/real_hand_l20_8_le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; visual mesh filename=package://real_hand_pybullet/urdf/meshes/real_hand_l20_8_le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
- link little_link1: geometry collision mesh filename=package://real_hand_pybullet/urdf/meshes/real_hand_l20_8_le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; visual mesh filename=package://real_hand_pybullet/urdf/meshes/real_hand_l20_8_le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
- link little_link2: geometry collision mesh filename=package://real_hand_pybullet/urdf/meshes/real_hand_l20_8_le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; visual mesh filename=package://real_hand_pybullet/urdf/meshes/real_hand_l20_8_le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
- link little_link3: geometry collision mesh filename=package://real_hand_pybullet/urdf/meshes/real_hand_l20_8_le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; visual mesh filename=package://real_hand_pybullet/urdf/meshes/real_hand_l20_8_le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
- link little_link4: geometry collision mesh filename=package://real_hand_pybullet/urdf/meshes/real_hand_l20_8_le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; visual mesh filename=package://real_hand_pybullet/urdf/meshes/real_hand_l20_8_le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
- link middle_link0: geometry collision mesh filename=package://real_hand_pybullet/urdf/meshes/real_hand_l20_8_le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; visual mesh filename=package://real_hand_pybullet/urdf/meshes/real_hand_l20_8_le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
- link middle_link1: geometry collision mesh filename=package://real_hand_pybullet/urdf/meshes/real_hand_l20_8_le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; visual mesh filename=package://real_hand_pybullet/urdf/meshes/real_hand_l20_8_le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
- link middle_link2: geometry collision mesh filename=package://real_hand_pybullet/urdf/meshes/real_hand_l20_8_le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; visual mesh filename=package://real_hand_pybullet/urdf/meshes/real_hand_l20_8_le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
- link middle_link3: geometry collision mesh filename=package://real_hand_pybullet/urdf/meshes/real_hand_l20_8_le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; visual mesh filename=package://real_hand_pybullet/urdf/meshes/real_hand_l20_8_le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
- link middle_link4: geometry collision mesh filename=package://real_hand_pybullet/urdf/meshes/real_hand_l20_8_le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; visual mesh filename=package://real_hand_pybullet/urdf/meshes/real_hand_l20_8_le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
- link ring_link0: geometry collision mesh filename=package://real_hand_pybullet/urdf/meshes/real_hand_l20_8_le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; visual mesh filename=package://real_hand_pybullet/urdf/meshes/real_hand_l20_8_le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
- link ring_link1: geometry collision mesh filename=package://real_hand_pybullet/urdf/meshes/real_hand_l20_8_le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; visual mesh filename=package://real_hand_pybullet/urdf/meshes/real_hand_l20_8_le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
- link ring_link2: geometry collision mesh filename=package://real_hand_pybullet/urdf/meshes/real_hand_l20_8_le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; visual mesh filename=package://real_hand_pybullet/urdf/meshes/real_hand_l20_8_le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
- link ring_link3: geometry collision mesh filename=package://real_hand_pybullet/urdf/meshes/real_hand_l20_8_le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; visual mesh filename=package://real_hand_pybullet/urdf/meshes/real_hand_l20_8_le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
- link ring_link4: geometry collision mesh filename=package://real_hand_pybullet/urdf/meshes/real_hand_l20_8_le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; visual mesh filename=package://real_hand_pybullet/urdf/meshes/real_hand_l20_8_le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
- link thumb_link0: geometry collision mesh filename=package://real_hand_pybullet/urdf/meshes/real_hand_l20_8_le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; visual mesh filename=package://real_hand_pybullet/urdf/meshes/real_hand_l20_8_le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
- link thumb_link1: geometry collision mesh filename=package://real_hand_pybullet/urdf/meshes/real_hand_l20_8_le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; visual mesh filename=package://real_hand_pybullet/urdf/meshes/real_hand_l20_8_le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
- link thumb_link2: geometry collision mesh filename=package://real_hand_pybullet/urdf/meshes/real_hand_l20_8_le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; visual mesh filename=package://real_hand_pybullet/urdf/meshes/real_hand_l20_8_le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
- link thumb_link3: geometry collision mesh filename=package://real_hand_pybullet/urdf/meshes/real_hand_l20_8_le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; visual mesh filename=package://real_hand_pybullet/urdf/meshes/real_hand_l20_8_le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
- link thumb_link4: geometry collision mesh filename=package://real_hand_pybullet/urdf/meshes/real_hand_l20_8_le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; visual mesh filename=package://real_hand_pybullet/urdf/meshes/real_hand_l20_8_le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
- link thumb_link5: geometry collision mesh filename=package://real_hand_pybullet/urdf/meshes/real_hand_l20_8_le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; visual mesh filename=package://real_hand_pybullet/urdf/meshes/real_hand_l20_8_le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

File: example/Linker_hand_Sapien/urdf/linker_hand_l20_8_right.urdf (robot description, URDF)
Before this commit: robot linkerhand_l20_8_right, 27 links, 26 joints
Links:
- link base_link: geometry collision mesh filename=meshes/real_hand_l20_8_right/base_link.STL; visual mesh filename=meshes/real_hand_l20_8_right/base_link.STL
- link index_link0: geometry collision mesh filename=meshes/real_hand_l20_8_right/index_link0.STL; visual mesh filename=meshes/real_hand_l20_8_right/index_link0.STL
- link index_link1: geometry collision mesh filename=meshes/real_hand_l20_8_right/index_link1.STL; visual mesh filename=meshes/real_hand_l20_8_right/index_link1.STL
- link index_link2: geometry collision mesh filename=meshes/real_hand_l20_8_right/index_link2.STL; visual mesh filename=meshes/real_hand_l20_8_right/index_link2.STL
- link index_link3: geometry collision mesh filename=meshes/real_hand_l20_8_right/index_link3.STL; visual mesh filename=meshes/real_hand_l20_8_right/index_link3.STL
- link index_link4: geometry collision mesh filename=meshes/real_hand_l20_8_right/index_link4.STL; visual mesh filename=meshes/real_hand_l20_8_right/index_link4.STL
- link little_link0: geometry collision mesh filename=meshes/real_hand_l20_8_right/little_link0.STL; visual mesh filename=meshes/real_hand_l20_8_right/little_link0.STL
- link little_link1: geometry collision mesh filename=meshes/real_hand_l20_8_right/little_link1.STL; visual mesh filename=meshes/real_hand_l20_8_right/little_link1.STL
- link little_link2: geometry collision mesh filename=meshes/real_hand_l20_8_right/little_link2.STL; visual mesh filename=meshes/real_hand_l20_8_right/little_link2.STL
- link little_link3: geometry collision mesh filename=meshes/real_hand_l20_8_right/little_link3.STL; visual mesh filename=meshes/real_hand_l20_8_right/little_link3.STL
- link little_link4: geometry collision mesh filename=meshes/real_hand_l20_8_right/little_link4.STL; visual mesh filename=meshes/real_hand_l20_8_right/little_link4.STL
- link middle_link0: geometry collision mesh filename=meshes/real_hand_l20_8_right/middle_link0.STL; visual mesh filename=meshes/real_hand_l20_8_right/middle_link0.STL
- link middle_link1: geometry collision mesh filename=meshes/real_hand_l20_8_right/middle_link1.STL; visual mesh filename=meshes/real_hand_l20_8_right/middle_link1.STL
- link middle_link2: geometry collision mesh filename=meshes/real_hand_l20_8_right/middle_link2.STL; visual mesh filename=meshes/real_hand_l20_8_right/middle_link2.STL
- link middle_link3: geometry collision mesh filename=meshes/real_hand_l20_8_right/middle_link3.STL; visual mesh filename=meshes/real_hand_l20_8_right/middle_link3.STL
- link middle_link4: geometry collision mesh filename=meshes/real_hand_l20_8_right/middle_link4.STL; visual mesh filename=meshes/real_hand_l20_8_right/middle_link4.STL
- link ring_link0: geometry collision mesh filename=meshes/real_hand_l20_8_right/ring_link0.STL; visual mesh filename=meshes/real_hand_l20_8_right/ring_link0.STL
- link ring_link1: geometry collision mesh filename=meshes/real_hand_l20_8_right/ring_link1.STL; visual mesh filename=meshes/real_hand_l20_8_right/ring_link1.STL
- link ring_link2: geometry collision mesh filename=meshes/real_hand_l20_8_right/ring_link2.STL; visual mesh filename=meshes/real_hand_l20_8_right/ring_link2.STL
- link ring_link3: geometry collision mesh filename=meshes/real_hand_l20_8_right/ring_link3.STL; visual mesh filename=meshes/real_hand_l20_8_right/ring_link3.STL
- link ring_link4: geometry collision mesh filename=meshes/real_hand_l20_8_right/ring_link4.STL; visual mesh filename=meshes/real_hand_l20_8_right/ring_link4.STL
- link thumb_link0: geometry collision mesh filename=meshes/real_hand_l20_8_right/thumb_link0.STL; visual mesh filename=meshes/real_hand_l20_8_right/thumb_link0.STL
- link thumb_link1: geometry collision mesh filename=meshes/real_hand_l20_8_right/thumb_link1.STL; visual mesh filename=meshes/real_hand_l20_8_right/thumb_link1.STL
- link thumb_link2: geometry collision mesh filename=meshes/real_hand_l20_8_right/thumb_link2.STL; visual mesh filename=meshes/real_hand_l20_8_right/thumb_link2.STL
- link thumb_link3: geometry collision mesh filename=meshes/real_hand_l20_8_right/thumb_link3.STL; visual mesh filename=meshes/real_hand_l20_8_right/thumb_link3.STL
- link thumb_link4: geometry collision mesh filename=meshes/real_hand_l20_8_right/thumb_link4.STL; visual mesh filename=meshes/real_hand_l20_8_right/thumb_link4.STL
- link thumb_link5: geometry collision mesh filename=meshes/real_hand_l20_8_right/thumb_link5.STL; visual mesh filename=meshes/real_hand_l20_8_right/thumb_link5.STL
